File: ATWCane-V0.kicad_pcb (KiCad board)
At the start: 2 copper layers, 27 parts, among them J1 Jack-DC, Q1 BD140, Q2 BD140, Q3 BD140, Q4 BD140, Q5 BD140, Q6 BD140, U1 HX711-board, U10 Solenoid, U11 MPU6050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

Commit message: Update ATWCane-V0.kicad_pcb
Parts:
- added J2: Jack-DC, ATWCane-sensor-stuff:Board outline V1, F.Cu at (91.0, 82.0)
- moved U8 123.0 mm to (65.0, 95.0)
- moved U9 123.0 mm to (65.0, 85.9)
- moved U10 116.8 mm to (65.0, 76.9)
- moved U11 79.4 mm to (87.9, 96.6)
- moved U2 77.9 mm to (71.4, 67.0)
- moved R8 37.8 mm to (139.2, 81.3)
- moved U5 29.9 mm to (86.0, 152.1)
- moved R7 22.4 mm to (110.2, 33.3)
Other:
- board outline added: 68.9 x 71.9 mm
Changed lines of the file:
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@@
   )
   (footprint "ATWCane-sensor-stuff:Solenoid" (layer "F.Cu")
-    (at 186.455 114.63)
+    (at 65 95)
     (property "Sheetfile" "ATWCane-V0.kicad_sch")
     (property "Sheetname" "")
@@
   )
   (footprint "footprints:810F4R0" (layer "F.Cu")
-    (at 101.826 87.192)
+    (at 139.172 81.27)
     (property "Sheetfile" "ATWCane-V0.kicad_sch")
     (property "Sheetname" "")
@@
     )
   )
+  (footprint "ATWCane-sensor-stuff:Board outline V1" (layer "F.Cu")
+    (at 91 82)
+    (property "Sheetfile" "ATWCane-V0.kicad_sch")
+    (property "Sheetname" "")
+    (attr through_hole)
+    (fp_text reference "J2" (at 0 -0.5 unlocked) (layer "F.SilkS")
+      (effects (font (size 1 1) (thickness 0.15)))
+    )
+    (fp_text value "Jack-DC" (at 0 1 unlocked) (layer "F.Fab")
+      (effects (font (size 1 1) (thickness 0.15)))
+    )
+    (fp_text user "${REFERENCE}" (at 0 2.5 unlocked) (layer "F.Fab")
+      (effects (font (size 1 1) (thickness 0.15)))
+    )
+    (fp_poly (pts
+        (xy 1.885416 -35.892198)
+        (xy 4.495901 -27.851027)
+        (xy 1.814863 -22.313905)
+        (xy 0.897665 -14.837026)
+        (xy 10.034365 -9.511516)
+        (xy 17.759985 -15.754003)
+        (xy 20.229361 -19.386637)
+        (xy 27.178892 -21.784881)
+        (xy 27.830067 -20.909443)
+        (xy 28.54133 -19.849474)
+        (xy 29.418419 -18.405187)
+        (xy 30.392864 -16.59947)
+        (xy 31.396195 -14.455208)
+        (xy 31.887297 -13.263274)
+        (xy 32.359944 -11.995287)
+        (xy 32.805577 -10.654107)
+        (xy 33.215639 -9.242595)
+        (xy 33.581571 -7.763612)
+        (xy 33.894813 -6.220018)
+        (xy 34.146807 -4.614675)
+        (xy 34.328995 -2.950443)
+        (xy 34.432818 -1.230183)
+        (xy 34.449717 0.543245)
+        (xy 34.371133 2.366979)
+        (xy 34.188509 4.238158)
+        (xy 33.893284 6.153923)
+        (xy 33.476901 8.111411)
+        (xy 32.9308 10.107762)
+        (xy 32.246424 12.140116)
+        (xy 31.415212 14.205611)
+        (xy 30.428608 16.301387)
+        (xy 29.278052 18.424583)
+        (xy 27.954985 20.572338)
+        (xy 19.98242 18.985264)
+        (xy 16.52529 13.906632)
+        (xy 10.528231 9.357025)
+        (xy 1.320982 14.576733)
+        (xy 2.802607 24.381321)
+        (xy 4.672278 28.366638)
+        (xy 2.626223 35.702446)
+        (xy 1.577564 35.83422)
+        (xy 0.342703 35.92586)
+        (xy -1.298324 35.969713)
+        (xy -3.294875 35.91706)
+        (xy -5.596308 35.719184)
+        (xy -8.151983 35.327366)
+        (xy -9.509336 35.043505)
+        (xy -10.911258 34.69289)
+        (xy -12.351419 34.26943)
+        (xy -13.82349 33.767037)
+        (xy -15.32114 33.17962)
+        (xy -16.838039 32.50109)
+        (xy -18.367857 31.725356)
+        (xy -19.904264 30.84633)
+        (xy -21.440928 29.857921)
+        (xy -22.971521 28.754041)
+        (xy -24.489712 27.528598)
+        (xy -25.989171 26.175503)
+        (xy -27.463567 24.688668)
+        (xy -28.906571 23.062001)
+        (xy -30.311852 21.289413)
+        (xy -31.67308 19.364815)
+        (xy -32.983924 17.282117)
+        (xy -34.238056 15.035229)
+        (xy -28.770148 8.722203)
+        (xy -22.631981 8.228447)
+        (xy -15.717724 5.265911)
+        (xy -15.717724 -5.314577)
+        (xy -24.995528 -8.841408)
+        (xy -29.369854 -9.158823)
+        (xy -34.449716 -14.237457)
+        (xy -33.999661 -15.233029)
+        (xy -33.418179 -16.37187)
+        (xy -32.582248 -17.844192)
+        (xy -31.479262 -19.579581)
+        (xy -30.096609 -21.507619)
+        (xy -28.421683 -23.557891)
+        (xy -27.470677 -24.606859)
+        (xy -26.441874 -25.65998)
+        (xy -25.333699 -26.708451)
+        (xy -24.144574 -27.743471)
+        (xy -22.872924 -28.756237)
+        (xy -21.517174 -29.737947)
+        (xy -20.075746 -30.679799)
+        (xy -18.547065 -31.572992)
+        (xy -16.929554 -32.408724)
+        (xy -15.221638 -33.178191)
+        (xy -13.421741 -33.872593)
+        (xy -11.528285 -34.483127)
+        (xy -9.539697 -35.000992)
+        (xy -7.454398 -35.417384)
+        (xy -5.270813 -35.723503)
+        (xy -2.987367 -35.910547)
+        (xy -0.602482 -35.969712)
+        (xy 1.885416 -35.892198)
+      ) (layer "Edge.Cuts") (width 0.352725) (fill solid))
+    (group "" (id c9b0f093-79f7-44a9-9a01-140d009dab54)
+      (members
+        95b9926a-6923-4d22-94a9-a7e0924d3712
+      )
+    )
+  )
   (footprint "Connector_PinHeader_2.54mm:PinHeader_1x03_P2.54mm_Vertical" (layer "F.Cu")
     (at 191.17 71.695)
@@
   )
   (footprint "Arduino:Arduino_Nano" (layer "F.Cu")
-    (at 148.994 73.959)
+    (at 71.38 66.95)
     (descr "Arduino Nano")
     (tags "Arduino Nano")
@@
   )
   (footprint "ATWCane-sensor-stuff:Solenoid" (layer "F.Cu")
-    (at 172.545 122.43)
+    (at 65 76.88)
     (property "Sheetfile" "ATWCane-V0.kicad_sch")
     (property "Sheetname" "")
@@
   )
   (footprint "ATWCane-sensor-stuff:Solenoid" (layer "F.Cu")
-    (at 186.455 105.51)
+    (at 65 85.88)
     (property "Sheetfile" "ATWCane-V0.kicad_sch")
     (property "Sheetname" "")
@@
   )
   (footprint "ATWCane-sensor-stuff:MPU6050" (layer "F.Cu")
-    (at 167.135 91.38)
+    (at 87.9 96.63)
     (property "Sheetfile" "ATWCane-V0.kicad_sch")
     (property "Sheetname" "")
@@
   )
   (footprint "footprints:810F4R0" (layer "F.Cu")
-    (at 101.826 54.092)
+    (at 110.172 33.27)
     (property "Sheetfile" "ATWCane-V0.kicad_sch")
     (property "Sheetname" "")
@@
   )
   (footprint "ATWCane-sensor-stuff:HX711board" (layer "F.Cu")
-    (at 102.915 127.5)
-    (property "Sheetfile" "ATWCane-V0.kicad_sch")
-    (property "Sheetname" "")
+    (at 86 152.14)
+    (property "Sheetfile" "ATWCane-V0.kicad_sch")
+    (property "Sheetname" "")

Commit message: Update ATWCane-V0.kicad_pcb
Parts:
- R1, R2, R3, R4, R5, R6: footprint Resistor_THT:R_Axial_DIN0207_L6.3mm_D2.5mm_P10.16mm_Horizontal -> Resistor_THT:R_Axial_DIN0207_L6.3mm_D2.5mm_P2.54mm_Vertical
- R9: value 810F4R0 -> Aluminum_Axiel_810_OHM
- moved Q1 189.8 mm to (73.4, 110.0), turned to 145 degrees
- moved Q2 174.2 mm to (62.1, 65.4), turned to 55 degrees
- moved Q4 163.3 mm to (73.1, 54.4), turned to 27.5 degrees
- moved R3 162.9 mm to (75.4, 107.4)
- moved U2 139.5 mm to (206.4, 102.0)
- moved U7 119.1 mm to (72.6, 60.7), turned to 115 degrees
- moved Q5 102.6 mm to (88.4, 114.1), turned to 175 degrees
- moved U6 98.1 mm to (70.6, 97.3), turned to -40 degrees
- moved J1 90.1 mm to (87.5, 46.0), turned to -90 degrees
- moved R6 82.8 mm to (63.8, 70.4)
- moved R1 76.2 mm to (68.8, 67.0), turned to 90 degrees
- moved Q6 73.3 mm to (117.6, 66.0), turned to -65 degrees
- moved R9 72.0 mm to (79.2, 64.8), turned to -47 degrees
- moved U3 71.8 mm to (117.5, 91.5), turned to -101.5 degrees
- moved U11 70.7 mm to (153.1, 124.1)
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
Commit message: Update ATWCane-V0.kicad_pcb
Parts:
- removed R7, R8: 810F4R0, footprints:810F4R0
- removed U1, U4, U5: HX711-board, ATWCane-sensor-stuff:HX711board
- removed U11: MPU6050, ATWCane-sensor-stuff:MPU6050
- removed U2: Arduino_Nano, Arduino:Arduino_Nano

Commit message: Update ATWCane-V0.kicad_pcb
Parts:
- added R7: 810F4R0, footprints:810F4R0, F.Cu at (153.0, 36.6)
- added R8: 810F4R0, footprints:810F4R0, F.Cu at (148.3, 67.4)
- added U1: HX711-board, ATWCane-sensor-stuff:HX711board, F.Cu at (200.1, 61.3)
- added U11: MPU6050, ATWCane-sensor-stuff:MPU6050, F.Cu at (153.1, 124.1)
- added U2: Arduino_Nano, Arduino:Arduino_Nano, F.Cu at (206.4, 102.0)
- added U4: HX711-board, ATWCane-sensor-stuff:HX711board, F.Cu at (200.1, 87.1)
- added U5: HX711-board, ATWCane-sensor-stuff:HX711board, F.Cu at (160.8, 165.4)
- moved J2 84.9 mm to (95.8, -2.73)
Other:
- board size 68.9 x 71.9 mm -> 153.1 x 114.5 mm
