File: ATWCane-V0.kicad_sch (KiCad schematic)
At the start: 27 parts, among them J1 Jack-DC, Q1 BD140, Q2 BD140, Q3 BD140, Q4 BD140, Q5 BD140, Q6 BD140, U1 HX711-board, U10 Solenoid, U11 MPU6050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

Commit message: Update ATWCane-V0.kicad_sch
Parts:
- added J?: Jack-DC, ATWCane-sensor-stuff:Board outline V1, symbol Connector:Jack-DC
Changed lines of the file:
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@@
     (pin "3")
+  )
+  (symbol (lib_id "Connector:Jack-DC") (at 103.0224 110.49 0) (unit 1)
+    (in_bom yes) (on_board yes) (fields_autoplaced)
+    (property "Reference" "J?" (id 0) (at 103.0224 101.6 0))
+    (property "Value" "Jack-DC" (id 1) (at 103.0224 104.14 0))
+    (property "Footprint" "ATWCane-sensor-stuff:Board outline V1" (id 2) (at 104.2924 111.506 0)
+      (effects (font (size 1.27 1.27)) hide)
+    )
+    (property "Datasheet" "~" (id 3) (at 104.2924 111.506 0)
+      (effects (font (size 1.27 1.27)) hide)
+    )
+    (pin "1")
+    (pin "2")
   )
   (symbol (lib_id "Device:R_US") (at 55.372 162.306 90) (unit 1)
@@
       (reference "J1") (unit 1) (value "Jack-DC") (footprint "Connector_BarrelJack:BarrelJack_Horizontal")
     )
+    (path "/e89e5b16-554a-4d97-8f95-fc89c9b40d74"
+      (reference "J?") (unit 1) (value "Jack-DC") (footprint "ATWCane-sensor-stuff:Board outline V1")
+    )
     (path "/5297ab3c-650b-4a41-a6f7-bd98c7dda8cb"

Commit message: Update ATWCane-V0.kicad_sch
Parts:
- R1, R2, R3, R4, R5, R6: footprint Resistor_THT:R_Axial_DIN0207_L6.3mm_D2.5mm_P10.16mm_Horizontal -> Resistor_THT:R_Axial_DIN0207_L6.3mm_D2.5mm_P2.54mm_Vertical
Changed lines of the file:
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@@
     (property "Reference" "R1" (id 0) (at 129.286 23.876 90))
     (property "Value" "1kΩ" (id 1) (at 125.476 23.876 90))
-    (property "Footprint" "Resistor_THT:R_Axial_DIN0207_L6.3mm_D2.5mm_P10.16mm_Horizontal" (id 2) (at 125.476 20.32 90)
+    (property "Footprint" "Resistor_THT:R_Axial_DIN0207_L6.3mm_D2.5mm_P2.54mm_Vertical" (id 2) (at 125.476 20.32 90)
       (effects (font (size 1.27 1.27)) hide)
     )
@@
     (property "Reference" "R4" (id 0) (at 59.69 170.688 90))
     (property "Value" "1kΩ" (id 1) (at 55.88 170.688 90))
-    (property "Footprint" "Resistor_THT:R_Axial_DIN0207_L6.3mm_D2.5mm_P10.16mm_Horizontal" (id 2) (at 55.88 167.132 90)
+    (property "Footprint" "Resistor_THT:R_Axial_DIN0207_L6.3mm_D2.5mm_P2.54mm_Vertical" (id 2) (at 55.88 167.132 90)
       (effects (font (size 1.27 1.27)) hide)
     )
@@
     (property "Reference" "R6" (id 0) (at 246.634 177.546 90))
     (property "Value" "1kΩ" (id 1) (at 250.444 177.546 90))
-    (property "Footprint" "Resistor_THT:R_Axial_DIN0207_L6.3mm_D2.5mm_P10.16mm_Horizontal" (id 2) (at 250.444 181.102 90)
+    (property "Footprint" "Resistor_THT:R_Axial_DIN0207_L6.3mm_D2.5mm_P2.54mm_Vertical" (id 2) (at 250.444 181.102 90)
       (effects (font (size 1.27 1.27)) hide)
     )
@@
     (property "Reference" "R5" (id 0) (at 246.38 171.704 90))
     (property "Value" "1kΩ" (id 1) (at 250.19 171.704 90))
-    (property "Footprint" "Resistor_THT:R_Axial_DIN0207_L6.3mm_D2.5mm_P10.16mm_Horizontal" (id 2) (at 250.19 175.26 90)
+    (property "Footprint" "Resistor_THT:R_Axial_DIN0207_L6.3mm_D2.5mm_P2.54mm_Vertical" (id 2) (at 250.19 175.26 90)
       (effects (font (size 1.27 1.27)) hide)
     )
@@
     (property "Reference" "R2" (id 0) (at 129.54 29.718 90))
     (property "Value" "1kΩ" (id 1) (at 125.73 29.718 90))
-    (property "Footprint" "Resistor_THT:R_Axial_DIN0207_L6.3mm_D2.5mm_P10.16mm_Horizontal" (id 2) (at 125.73 26.162 90)
+    (property "Footprint" "Resistor_THT:R_Axial_DIN0207_L6.3mm_D2.5mm_P2.54mm_Vertical" (id 2) (at 125.73 26.162 90)
       (effects (font (size 1.27 1.27)) hide)
     )
@@
     (property "Reference" "R3" (id 0) (at 59.436 164.846 90))
     (property "Value" "1kΩ" (id 1) (at 55.626 164.846 90))
-    (property "Footprint" "Resistor_THT:R_Axial_DIN0207_L6.3mm_D2.5mm_P10.16mm_Horizontal" (id 2) (at 55.626 161.29 90)
+    (property "Footprint" "Resistor_THT:R_Axial_DIN0207_L6.3mm_D2.5mm_P2.54mm_Vertical" (id 2) (at 55.626 161.29 90)
       (effects (font (size 1.27 1.27)) hide)
     )
@@
     )
     (path "/1b495a70-83a2-4dbe-8b8b-5d9ee3fbd1ac"
-      (reference "R1") (unit 1) (value "1kΩ") (footprint "Resistor_THT:R_Axial_DIN0207_L6.3mm_D2.5mm_P10.16mm_Horizontal")
+      (reference "R1") (unit 1) (value "1kΩ") (footprint "Resistor_THT:R_Axial_DIN0207_L6.3mm_D2.5mm_P2.54mm_Vertical")
     )
     (path "/90cc22e9-ce1b-422f-8bca-d0423a0a0560"
-      (reference "R2") (unit 1) (value "1kΩ") (footprint "Resistor_THT:R_Axial_DIN0207_L6.3mm_D2.5mm_P10.16mm_Horizontal")
+      (reference "R2") (unit 1) (value "1kΩ") (footprint "Resistor_THT:R_Axial_DIN0207_L6.3mm_D2.5mm_P2.54mm_Vertical")
     )
     (path "/f47b4767-5cec-4986-bec1-5310f9f880e9"
-      (reference "R3") (unit 1) (value "1kΩ") (footprint "Resistor_THT:R_Axial_DIN0207_L6.3mm_D2.5mm_P10.16mm_Horizontal")
+      (reference "R3") (unit 1) (value "1kΩ") (footprint "Resistor_THT:R_Axial_DIN0207_L6.3mm_D2.5mm_P2.54mm_Vertical")
     )
     (path "/51a12b73-e8c3-4ae9-bbe2-1299363a5a15"
-      (reference "R4") (unit 1) (value "1kΩ") (footprint "Resistor_THT:R_Axial_DIN0207_L6.3mm_D2.5mm_P10.16mm_Horizontal")
+      (reference "R4") (unit 1) (value "1kΩ") (footprint "Resistor_THT:R_Axial_DIN0207_L6.3mm_D2.5mm_P2.54mm_Vertical")
     )
     (path "/774fbced-0a0d-4665-8e8f-f2621360dee9"
-      (reference "R5") (unit 1) (value "1kΩ") (footprint "Resistor_THT:R_Axial_DIN0207_L6.3mm_D2.5mm_P10.16mm_Horizontal")
+      (reference "R5") (unit 1) (value "1kΩ") (footprint "Resistor_THT:R_Axial_DIN0207_L6.3mm_D2.5mm_P2.54mm_Vertical")
     )
     (path "/6f4d0bf4-c152-4d2e-946b-61ac7345f8b4"
-      (reference "R6") (unit 1) (value "1kΩ") (footprint "Resistor_THT:R_Axial_DIN0207_L6.3mm_D2.5mm_P10.16mm_Horizontal")
+      (reference "R6") (unit 1) (value "1kΩ") (footprint "Resistor_THT:R_Axial_DIN0207_L6.3mm_D2.5mm_P2.54mm_Vertical")
     )
     (path "/4861ac2f-8d8c-4811-9567-2a97a88d31e0"

Commit message: Update ATWCane-V0.kicad_sch
Parts:
- gave numbers to parts that had none: 1
Changed lines of the file:
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@@
   (symbol (lib_id "Connector:Jack-DC") (at 103.0224 110.49 0) (unit 1)
     (in_bom yes) (on_board yes) (fields_autoplaced)
-    (property "Reference" "J?" (id 0) (at 103.0224 101.6 0))
+    (property "Reference" "J2" (id 0) (at 103.0224 101.6 0))
     (property "Value" "Jack-DC" (id 1) (at 103.0224 104.14 0))
     (property "Footprint" "ATWCane-sensor-stuff:Board outline V1" (id 2) (at 104.2924 111.506 0)
@@
     )
     (path "/e89e5b16-554a-4d97-8f95-fc89c9b40d74"
-      (reference "J?") (unit 1) (value "Jack-DC") (footprint "ATWCane-sensor-stuff:Board outline V1")
+      (reference "J2") (unit 1) (value "Jack-DC") (footprint "ATWCane-sensor-stuff:Board outline V1")
     )
     (path "/5297ab3c-650b-4a41-a6f7-bd98c7dda8cb"
